Commit message: Refactor, add odom and tf pub, add bumper

File: sjtu_drone_description/urdf/sjtu_drone.urdf.xacro (robot description, xacro)
@@ -68,4 +68,5 @@
       </ros>
       <bodyName>base_link</bodyName>
+      <pub_odom>true</pub_odom>
       <rollpitchProportionalGain>${mp['rollpitchProportionalGain']}</rollpitchProportionalGain>
       <rollpitchDifferentialGain>${mp['rollpitchDifferentialGain']}</rollpitchDifferentialGain>
@@ -108,9 +109,9 @@
           <rate>
             <mean> 0 </mean>
-            <stddev> 0 </stddev>
+            <stddev> 0.01 </stddev>
           </rate>
           <accel>
             <mean> 0 </mean>
-            <stddev> 0.00 </stddev>
+            <stddev> 0.01 </stddev>
           </accel>
         </noise>
@@ -119,4 +120,5 @@
         <ros>
           <namespace>${mp['namespace']}</namespace>
+          <!-- <remapping>imu:=imu</remapping> -->
         </ros>
         <initial_orientation_as_reference>false</initial_orientation_as_reference>
@@ -187,5 +189,5 @@
           <type>gaussian</type>
           <mean>0.0</mean>
-          <stddev>0.005</stddev>
+          <stddev>0.01</stddev>
         </noise>
       </camera>
@@ -222,5 +224,5 @@
           <type>gaussian</type>
           <mean>0.0</mean>
-          <stddev>0.005</stddev>
+          <stddev>0.01</stddev>
         </noise>
       </camera>
@@ -266,3 +268,19 @@
     </sensor>
   </gazebo>
+  <gazebo reference="base_link">
+    <sensor name="collision_sensor" type="contact">
+      <update_rate>100.0</update_rate>
+      <always_on>true</always_on>
+      <contact>
+        <collision>base_footprint_fixed_joint_lump__sjtu_drone_collision_collision</collision>
+      </contact>
+      <plugin name="collision_plugin" filename="libgazebo_ros_bumper.so">
+        <ros>
+          <namespace>${mp['namespace']}</namespace>
+          <!-- <remapping>bumper_states:=bumper_states</remapping> -->
+        </ros>
+        <frame_name>${mp['namespace']}/base_link</frame_name>
+      </plugin>
+    </sensor>
+  </gazebo>
 </robot>
